Commit message: Update URDF and rviz config

File: src/simple_bot_bringup/urdf/simple_bot.xacro (robot description, xacro)
@@ -48,5 +48,5 @@
         <parent link="base_link" />
         <child link="right_wheel_link" />
-        <origin xyz="0.2 ${(base_width/2) + (wheel_radius/2)} 0" rpy="0 0 0" />
+        <origin xyz="-0.2 ${(base_width/2) + (wheel_radius/2)} 0" rpy="0 0 0" />
         <axis xyz="1 0 0" />
         <limit velocity="1" effort="1" lower="-0.4" upper="0.04" />
@@ -77,5 +77,5 @@
         <parent link="base_link" />
         <child link="left_wheel_link" />
-        <origin xyz="-0.2 ${(base_width/2) + (wheel_radius/2)} 0" rpy="0 0 0" />
+        <origin xyz="0.2 ${(base_width/2) + (wheel_radius/2)} 0" rpy="0 0 0" />
     </joint>
 </robot>
